Commit message: feat(as2-piper): add RGB-D/3D-LiDAR sensor suite, proximity 4-door opener, ROS2 sim2real pkg, and RL fixes
- Add AS2 onboard sensor mounts (front_camera, lidar_link with non-occluding visual offset) to as2_piper.urdf/.xacro and Isaac Lab/OmniGraph ROS 2 sensor suite (as2_sensors.py) publishing RGB, metric Depth, CameraInfo, 3D PointCloud2, LaserScan, TF, and Clock
- Fix symmetric gripper jaws (link7/link8), FL_calf geometry, hospital_door.usda degree limits, standalone PiPER fixed root, and deterministic 48-D / 64-D RL joint ordering (preserve_order=True) with dynamic arm swing MDP events
- Implement simultaneous WASD + 6-DoF PiPER teleop and Key '1' proximity-gated (0.28m~0.90m, <=60 deg) automatic door opener across 4 hospital door mechanisms (lever_push, lever_pull, sliding, push_bar)
- Add ROS 2 Humble bringup package (as2_piper_bringup) with RGB-D/LiDAR door & handle detector, ONNX whole-body Sim-to-Real bridge with state liveness watchdog and latched handle propagation
- Add quantitative benchmark/ablation evaluator (evaluate_loco_manipulation.py), preflight checker, training runbook, LF shell script hygiene, and 21-test offline audit suite

File: robot_arms/piper/descriptions/as2_piper.urdf (robot description, URDF)
Before this commit: robot as2_piper, 11 links, 10 joints
Links:
- added link FL_calf, mass 0.154; collision cylinder length=0.12 radius=0.013; visual cylinder length=0.12 radius=0.013
- added link FL_calf_rotor, mass 0.089
- added link FL_calflower; collision cylinder length=0.065 radius=0.011
- added link FL_calflower1; collision cylinder length=0.03 radius=0.0155
- added link FL_foot, mass 0.04; collision sphere radius=0.022; visual sphere radius=0.022
- added link FL_hip, mass 0.678; collision cylinder length=0.04 radius=0.046; visual cylinder length=0.04 radius=0.046
- added link FL_hip_rotor, mass 0.089
- added link FL_thigh, mass 1.152; collision box size=0.213 0.0245 0.034; visual box size=0.213 0.0245 0.034
- added link FL_thigh_rotor, mass 0.089
- added link FR_calf, mass 0.154; collision cylinder length=0.12 radius=0.013; visual cylinder length=0.12 radius=0.013
- added link FR_calf_rotor, mass 0.089
- added link FR_calflower; collision cylinder length=0.065 radius=0.011
- added link FR_calflower1; collision cylinder length=0.03 radius=0.0155
- added link FR_foot, mass 0.04; collision sphere radius=0.022; visual sphere radius=0.022
- added link FR_hip, mass 0.678; collision cylinder length=0.04 radius=0.046; visual cylinder length=0.04 radius=0.046
- added link FR_hip_rotor, mass 0.089
- added link FR_thigh, mass 1.152; collision box size=0.213 0.0245 0.034; visual box size=0.213 0.0245 0.034
- added link FR_thigh_rotor, mass 0.089
- added link RL_calf, mass 0.154; collision cylinder length=0.12 radius=0.013; visual cylinder length=0.12 radius=0.013
- added link RL_calf_rotor, mass 0.089
- added link RL_calflower; collision cylinder length=0.065 radius=0.011
- added link RL_calflower1; collision cylinder length=0.03 radius=0.0155
- added link RL_foot, mass 0.04; collision sphere radius=0.022; visual sphere radius=0.022
- added link RL_hip, mass 0.678; collision cylinder length=0.04 radius=0.046; visual cylinder length=0.04 radius=0.046
- added link RL_hip_rotor, mass 0.089
- added link RL_thigh, mass 1.152; collision box size=0.213 0.0245 0.034; visual box size=0.213 0.0245 0.034
- added link RL_thigh_rotor, mass 0.089
- added link RR_calf, mass 0.154; collision cylinder length=0.12 radius=0.013; visual cylinder length=0.12 radius=0.013
- added link RR_calf_rotor, mass 0.089
- added link RR_calflower; collision cylinder length=0.065 radius=0.011
- added link RR_calflower1; collision cylinder length=0.03 radius=0.0155
- added link RR_foot, mass 0.04; collision sphere radius=0.022; visual sphere radius=0.022
- added link RR_hip, mass 0.678; collision cylinder length=0.04 radius=0.046; visual cylinder length=0.04 radius=0.046
- added link RR_hip_rotor, mass 0.089
- added link RR_thigh, mass 1.152; collision box size=0.213 0.0245 0.034; visual box size=0.213 0.0245 0.034
- added link RR_thigh_rotor, mass 0.089
- added link front_camera, mass 0.072; visual box size=0.025 0.090 0.025
- added link imu, mass 0.01
- added link lidar_link, mass 0.18; visual cylinder length=0.040 radius=0.032
- added link radar, mass 0.01
- link link7: geometry collision box size=0.015 0.05 0.01; visual box size=0.015 0.05 0.01
- link link8: geometry collision box size=0.015 0.05 0.01; visual box size=0.015 0.05 0.01
Joints:
- added joint FL_calf_joint: type revolute, parent FL_thigh, child FL_calf, origin xyz=0 0 -0.213 rpy=0 0 0, axis 0 1 0, limit lower=-2.7227 upper=-0.83776 effort=95.0 velocity=15.70
- added joint FL_calf_rotor_joint: type fixed, parent FL_thigh, child FL_calf_rotor, origin xyz=0 -0.03235 0 rpy=0 0 0
- added joint FL_calflower1_joint: type fixed, parent FL_calflower, child FL_calflower1, origin xyz=-0.01 0 -0.04 rpy=0 0.48 0
- added joint FL_calflower_joint: type fixed, parent FL_calf, child FL_calflower, origin xyz=0.020 0 -0.148 rpy=0 0.05 0
- added joint FL_foot_joint: type fixed, parent FL_calf, child FL_foot, origin xyz=0 0 -0.213 rpy=0 0 0
- added joint FL_hip_joint: type revolute, parent base, child FL_hip, origin xyz=0.1934 0.0465 0 rpy=0 0 0, axis 1 0 0, limit lower=-1.0472 upper=1.0472 effort=95.0 velocity=30.1
- added joint FL_hip_rotor_joint: type fixed, parent base, child FL_hip_rotor, origin xyz=0.11215 0.04675 0 rpy=0 0 0
- added joint FL_thigh_joint: type revolute, parent FL_hip, child FL_thigh, origin xyz=0 0.0955 0 rpy=0 0 0, axis 0 1 0, limit lower=-1.5708 upper=3.4907 effort=95.0 velocity=30.1
- added joint FL_thigh_rotor_joint: type fixed, parent FL_hip, child FL_thigh_rotor, origin xyz=0 -0.00015 0 rpy=0 0 0
- added joint FR_calf_joint: type revolute, parent FR_thigh, child FR_calf, origin xyz=0 0 -0.213 rpy=0 0 0, axis 0 1 0, limit lower=-2.7227 upper=-0.83776 effort=95.0 velocity=15.70
- added joint FR_calf_rotor_joint: type fixed, parent FR_thigh, child FR_calf_rotor, origin xyz=0 0.03235 0 rpy=0 0 0
- added joint FR_calflower1_joint: type fixed, parent FR_calflower, child FR_calflower1, origin xyz=-0.01 0 -0.04 rpy=0 0.48 0
- added joint FR_calflower_joint: type fixed, parent FR_calf, child FR_calflower, origin xyz=0.020 0 -0.148 rpy=0 0.05 0
- added joint FR_foot_joint: type fixed, parent FR_calf, child FR_foot, origin xyz=0 0 -0.213 rpy=0 0 0
- added joint FR_hip_joint: type revolute, parent base, child FR_hip, origin xyz=0.1934 -0.0465 0 rpy=0 0 0, axis 1 0 0, limit lower=-1.0472 upper=1.0472 effort=95.0 velocity=30.1
- added joint FR_hip_rotor_joint: type fixed, parent base, child FR_hip_rotor, origin xyz=0.11215 -0.04675 0 rpy=0 0 0
- added joint FR_thigh_joint: type revolute, parent FR_hip, child FR_thigh, origin xyz=0 -0.0955 0 rpy=0 0 0, axis 0 1 0, limit lower=-1.5708 upper=3.4907 effort=95.0 velocity=30.1
- added joint FR_thigh_rotor_joint: type fixed, parent FR_hip, child FR_thigh_rotor, origin xyz=0 0.00015 0 rpy=0 0 0
- added joint RL_calf_joint: type revolute, parent RL_thigh, child RL_calf, origin xyz=0 0 -0.213 rpy=0 0 0, axis 0 1 0, limit lower=-2.7227 upper=-0.83776 effort=95.0 velocity=15.70
- added joint RL_calf_rotor_joint: type fixed, parent RL_thigh, child RL_calf_rotor, origin xyz=0 -0.03235 0 rpy=0 0 0
- added joint RL_calflower1_joint: type fixed, parent RL_calflower, child RL_calflower1, origin xyz=-0.01 0 -0.04 rpy=0 0.48 0
- added joint RL_calflower_joint: type fixed, parent RL_calf, child RL_calflower, origin xyz=0.020 0 -0.148 rpy=0 0.05 0
- added joint RL_foot_joint: type fixed, parent RL_calf, child RL_foot, origin xyz=0 0 -0.213 rpy=0 0 0
- added joint RL_hip_joint: type revolute, parent base, child RL_hip, origin xyz=-0.1934 0.0465 0 rpy=0 0 0, axis 1 0 0, limit lower=-1.0472 upper=1.0472 effort=95.0 velocity=30.1
- added joint RL_hip_rotor_joint: type fixed, parent base, child RL_hip_rotor, origin xyz=-0.11215 0.04675 0 rpy=0 0 0
- added joint RL_thigh_joint: type revolute, parent RL_hip, child RL_thigh, origin xyz=0 0.0955 0 rpy=0 0 0, axis 0 1 0, limit lower=-0.5236 upper=4.5379 effort=95.0 velocity=30.1
- added joint RL_thigh_rotor_joint: type fixed, parent RL_hip, child RL_thigh_rotor, origin xyz=0 -0.00015 0 rpy=0 0 0
- added joint RR_calf_joint: type revolute, parent RR_thigh, child RR_calf, origin xyz=0 0 -0.213 rpy=0 0 0, axis 0 1 0, limit lower=-2.7227 upper=-0.83776 effort=95.0 velocity=15.70
- added joint RR_calf_rotor_joint: type fixed, parent RR_thigh, child RR_calf_rotor, origin xyz=0 0.03235 0 rpy=0 0 0
- added joint RR_calflower1_joint: type fixed, parent RR_calflower, child RR_calflower1, origin xyz=-0.01 0 -0.04 rpy=0 0.48 0
- added joint RR_calflower_joint: type fixed, parent RR_calf, child RR_calflower, origin xyz=0.020 0 -0.148 rpy=0 0.05 0
- added joint RR_foot_joint: type fixed, parent RR_calf, child RR_foot, origin xyz=0 0 -0.213 rpy=0 0 0
- added joint RR_hip_joint: type revolute, parent base, child RR_hip, origin xyz=-0.1934 -0.0465 0 rpy=0 0 0, axis 1 0 0, limit lower=-1.0472 upper=1.0472 effort=95.0 velocity=30.1
- added joint RR_hip_rotor_joint: type fixed, parent base, child RR_hip_rotor, origin xyz=-0.11215 -0.04675 0 rpy=0 0 0
- added joint RR_thigh_joint: type revolute, parent RR_hip, child RR_thigh, origin xyz=0 -0.0955 0 rpy=0 0 0, axis 0 1 0, limit lower=-0.5236 upper=4.5379 effort=95.0 velocity=30.1
- added joint RR_thigh_rotor_joint: type fixed, parent RR_hip, child RR_thigh_rotor, origin xyz=0 0.00015 0 rpy=0 0 0
- added joint front_camera_joint: type fixed, parent base, child front_camera, origin xyz=0.30 0.0 0.10 rpy=0 0 0
- added joint imu_joint: type fixed, parent base, child imu, origin xyz=-0.02557 0 0.04232 rpy=0 0 0
- added joint lidar_joint: type fixed, parent base, child lidar_link, origin xyz=0.285 0.0 0.045 rpy=0 0 0
- added joint radar_joint: type fixed, parent base, child radar, origin xyz=0.28945 0 -0.046825 rpy=0 2.8782 0
- joint joint1: limit lower=-2.618 upper=2.168 effort=100 velocity=5.0 -> lower=-2.618 upper=2.168 effort=100.0 velocity=5.0
- joint joint2: limit lower=0.0 upper=3.14 effort=100 velocity=5.0 -> lower=0.0 upper=3.14 effort=100.0 velocity=5.0
- joint joint3: limit lower=-2.967 upper=0.0 effort=100 velocity=5.0 -> lower=-2.967 upper=0.0 effort=100.0 velocity=5.0
- joint joint4: limit lower=-1.745 upper=1.745 effort=100 velocity=5.0 -> lower=-1.745 upper=1.745 effort=100.0 velocity=5.0
- joint joint5: limit lower=-1.22 upper=1.22 effort=100 velocity=5.0 -> lower=-1.22 upper=1.22 effort=100.0 velocity=5.0
- joint joint6: limit lower=-2.0944 upper=2.0944 effort=100 velocity=3.0 -> lower=-2.0944 upper=2.0944 effort=100.0 velocity=3.0
