Commit message: feat(as2-piper): add RGB-D/3D-LiDAR sensor suite, proximity 4-door opener, ROS2 sim2real pkg, and RL fixes
- Add AS2 onboard sensor mounts (front_camera, lidar_link with non-occluding visual offset) to as2_piper.urdf/.xacro and Isaac Lab/OmniGraph ROS 2 sensor suite (as2_sensors.py) publishing RGB, metric Depth, CameraInfo, 3D PointCloud2, LaserScan, TF, and Clock
- Fix symmetric gripper jaws (link7/link8), FL_calf geometry, hospital_door.usda degree limits, standalone PiPER fixed root, and deterministic 48-D / 64-D RL joint ordering (preserve_order=True) with dynamic arm swing MDP events
- Implement simultaneous WASD + 6-DoF PiPER teleop and Key '1' proximity-gated (0.28m~0.90m, <=60 deg) automatic door opener across 4 hospital door mechanisms (lever_push, lever_pull, sliding, push_bar)
- Add ROS 2 Humble bringup package (as2_piper_bringup) with RGB-D/LiDAR door & handle detector, ONNX whole-body Sim-to-Real bridge with state liveness watchdog and latched handle propagation
- Add quantitative benchmark/ablation evaluator (evaluate_loco_manipulation.py), preflight checker, training runbook, LF shell script hygiene, and 21-test offline audit suite

File: robot_arms/piper/descriptions/as2_piper.urdf.xacro (robot description, xacro)
@@ -4,4 +4,5 @@
   <!-- Unitree AS2 Industrial Quadruped Robot with AgileX PiPER Robotic Arm -->
   <!-- Computer Graphics and Vision Lab (CGV) - Isaac Sim 6.2.0 Integration  -->
+  <!-- Unified 20-DOF Mobile Manipulator Model                              -->
   <!-- ===================================================================== -->
   <!-- Parameters -->
@@ -67,5 +68,5 @@
     <child link="link1"/>
     <axis xyz="0 0 1"/>
-    <limit lower="-2.618" upper="2.168" effort="100" velocity="5.0"/>
+    <limit lower="-2.618" upper="2.168" effort="100.0" velocity="5.0"/>
   </joint>
   <link name="link1">
@@ -97,5 +98,5 @@
     <child link="link2"/>
     <axis xyz="0 0 1"/>
-    <limit lower="0.0" upper="3.14" effort="100" velocity="5.0"/>
+    <limit lower="0.0" upper="3.14" effort="100.0" velocity="5.0"/>
   </joint>
   <link name="link2">
@@ -125,5 +126,5 @@
     <child link="link3"/>
     <axis xyz="0 0 1"/>
-    <limit lower="-2.967" upper="0.0" effort="100" velocity="5.0"/>
+    <limit lower="-2.967" upper="0.0" effort="100.0" velocity="5.0"/>
   </joint>
   <link name="link3">
@@ -153,5 +154,5 @@
     <child link="link4"/>
     <axis xyz="0 0 1"/>
-    <limit lower="-1.745" upper="1.745" effort="100" velocity="5.0"/>
+    <limit lower="-1.745" upper="1.745" effort="100.0" velocity="5.0"/>
   </joint>
   <link name="link4">
@@ -181,5 +182,5 @@
     <child link="link5"/>
     <axis xyz="0 0 1"/>
-    <limit lower="-1.22" upper="1.22" effort="100" velocity="5.0"/>
+    <limit lower="-1.22" upper="1.22" effort="100.0" velocity="5.0"/>
   </joint>
   <link name="link5">
@@ -209,5 +210,5 @@
     <child link="link6"/>
     <axis xyz="0 0 1"/>
-    <limit lower="-2.0944" upper="2.0944" effort="100" velocity="3.0"/>
+    <limit lower="-2.0944" upper="2.0944" effort="100.0" velocity="3.0"/>
   </joint>
   <link name="link6">
@@ -267,19 +268,19 @@
   <link name="link7">
     <inertial>
-      <origin xyz="0 0 0.02" rpy="0 0 0"/>
+      <origin xyz="0 0.025 0" rpy="0 0 0"/>
       <mass value="0.05"/>
-      <inertia ixx="0.00005" ixy="0" ixz="0" iyy="0.00005" iyz="0" izz="0.00002"/>
-    </inertial>
-    <visual>
-      <origin xyz="0 0 0.02" rpy="0 0 0"/>
-      <geometry>
-        <box size="0.015 0.01 0.04"/>
-      </geometry>
-      <material name="matte_black"/>
-    </visual>
-    <collision>
-      <origin xyz="0 0 0.02" rpy="0 0 0"/>
-      <geometry>
-        <box size="0.015 0.01 0.04"/>
+      <inertia ixx="0.00005" ixy="0" ixz="0" iyy="0.00002" iyz="0" izz="0.00005"/>
+    </inertial>
+    <visual>
+      <origin xyz="0 0.025 0" rpy="0 0 0"/>
+      <geometry>
+        <box size="0.015 0.05 0.01"/>
+      </geometry>
+      <material name="matte_black"/>
+    </visual>
+    <collision>
+      <origin xyz="0 0.025 0" rpy="0 0 0"/>
+      <geometry>
+        <box size="0.015 0.05 0.01"/>
       </geometry>
     </collision>
@@ -295,21 +296,470 @@
   <link name="link8">
     <inertial>
-      <origin xyz="0 0 0.02" rpy="0 0 0"/>
+      <origin xyz="0 0.025 0" rpy="0 0 0"/>
       <mass value="0.05"/>
-      <inertia ixx="0.00005" ixy="0" ixz="0" iyy="0.00005" iyz="0" izz="0.00002"/>
-    </inertial>
-    <visual>
-      <origin xyz="0 0 0.02" rpy="0 0 0"/>
-      <geometry>
-        <box size="0.015 0.01 0.04"/>
-      </geometry>
-      <material name="matte_black"/>
-    </visual>
-    <collision>
-      <origin xyz="0 0 0.02" rpy="0 0 0"/>
-      <geometry>
-        <box size="0.015 0.01 0.04"/>
-      </geometry>
-    </collision>
-  </link>
+      <inertia ixx="0.00005" ixy="0" ixz="0" iyy="0.00002" iyz="0" izz="0.00005"/>
+    </inertial>
+    <visual>
+      <origin xyz="0 0.025 0" rpy="0 0 0"/>
+      <geometry>
+        <box size="0.015 0.05 0.01"/>
+      </geometry>
+      <material name="matte_black"/>
+    </visual>
+    <collision>
+      <origin xyz="0 0.025 0" rpy="0 0 0"/>
+      <geometry>
+        <box size="0.015 0.05 0.01"/>
+      </geometry>
+    </collision>
+  </link>
+  <!-- ===================================================================== -->
+  <!-- Unitree AS2 Industrial Quadruped Legs (12 DOF, 95 N.m Peak Torque)   -->
+  <!-- ===================================================================== -->
+  <!-- FL Leg -->
+  <link name="FL_hip">
+    <inertial>
+      <origin xyz="-0.0054 0.00194 -0.000105" rpy="0 0 0"/>
+      <mass value="0.678"/>
+      <inertia ixx="0.00048" ixy="-3.01E-06" ixz="1.11E-06" iyy="0.000884" iyz="-1.42E-06" izz="0.000596"/>
+    </inertial>
+    <visual>
+      <origin xyz="0 0.08 0" rpy="1.5707963 0 0"/>
+      <geometry><cylinder length="0.04" radius="0.046"/></geometry>
+      <material name="matte_black"/>
+    </visual>
+    <collision>
+      <origin xyz="0 0.08 0" rpy="1.5707963 0 0"/>
+      <geometry><cylinder length="0.04" radius="0.046"/></geometry>
+    </collision>
+  </link>
+  <joint name="FL_hip_joint" type="revolute">
+    <origin xyz="0.1934 0.0465 0" rpy="0 0 0"/>
+    <parent link="base"/>
+    <child link="FL_hip"/>
+    <axis xyz="1 0 0"/>
+    <limit lower="-1.0472" upper="1.0472" effort="95.0" velocity="30.1"/>
+  </joint>
+  <link name="FL_hip_rotor">
+    <inertial>
+      <origin xyz="0 0 0" rpy="0 0 0"/><mass value="0.089"/>
+      <inertia ixx="0.0001118" ixy="0" ixz="0" iyy="0.0000596" iyz="0" izz="0.0000596"/>
+    </inertial>
+  </link>
+  <joint name="FL_hip_rotor_joint" type="fixed">
+    <origin xyz="0.11215 0.04675 0" rpy="0 0 0"/>
+    <parent link="base"/><child link="FL_hip_rotor"/>
+  </joint>
+  <link name="FL_thigh">
+    <inertial>
+      <origin xyz="-0.00374 -0.0223 -0.0327" rpy="0 0 0"/>
+      <mass value="1.152"/>
+      <inertia ixx="0.00584" ixy="8.72E-05" ixz="-0.000289" iyy="0.0058" iyz="0.000808" izz="0.00103"/>
+    </inertial>
+    <visual>
+      <origin xyz="0 0 -0.1065" rpy="0 1.5707963 0"/>
+      <geometry><box size="0.213 0.0245 0.034"/></geometry>
+      <material name="matte_black"/>
+    </visual>
+    <collision>
+      <origin xyz="0 0 -0.1065" rpy="0 1.5707963 0"/>
+      <geometry><box size="0.213 0.0245 0.034"/></geometry>
+    </collision>
+  </link>
+  <joint name="FL_thigh_joint" type="revolute">
+    <origin xyz="0 0.0955 0" rpy="0 0 0"/>
+    <parent link="FL_hip"/><child link="FL_thigh"/>
+    <axis xyz="0 1 0"/>
+    <limit lower="-1.5708" upper="3.4907" effort="95.0" velocity="30.1"/>
+  </joint>
+  <link name="FL_thigh_rotor">
+    <inertial>
+      <origin xyz="0 0 0" rpy="0 0 0"/><mass value="0.089"/>
+      <inertia ixx="0.0000596" ixy="0" ixz="0" iyy="0.0001118" iyz="0" izz="0.0000596"/>
+    </inertial>
+  </link>
+  <joint name="FL_thigh_rotor_joint" type="fixed">
+    <origin xyz="0 -0.00015 0" rpy="0 0 0"/>
+    <parent link="FL_hip"/><child link="FL_thigh_rotor"/>
+  </joint>
+  <link name="FL_calf">
+    <inertial>
+      <origin xyz="0.00548 -0.000975 -0.115" rpy="0 0 0"/>
+      <mass value="0.154"/>
+      <inertia ixx="0.00108" ixy="3.4E-07" ixz="1.72E-05" iyy="0.0011" iyz="8.28E-06" izz="3.29E-05"/>
+    </inertial>
+    <visual>
+      <origin xyz="0.01 0 -0.06" rpy="0 -0.2 0"/>
+      <geometry><cylinder length="0.12" radius="0.013"/></geometry>
+      <material name="metallic"/>
+    </visual>
+    <collision>
+      <origin xyz="0.01 0 -0.06" rpy="0 -0.2 0"/>
+      <geometry><cylinder length="0.12" radius="0.013"/></geometry>
+    </collision>
+  </link>
+  <joint name="FL_calf_joint" type="revolute">
+    <origin xyz="0 0 -0.213" rpy="0 0 0"/>
+    <parent link="FL_thigh"/><child link="FL_calf"/>
+    <axis xyz="0 1 0"/>
+    <limit lower="-2.7227" upper="-0.83776" effort="95.0" velocity="15.70"/>
+  </joint>
+  <link name="FL_calflower">
+    <collision><origin xyz="0 0 0"/><geometry><cylinder length="0.065" radius="0.011"/></geometry></collision>
+  </link>
+  <joint name="FL_calflower_joint" type="fixed">
+    <origin xyz="0.020 0 -0.148" rpy="0 0.05 0"/>
+    <parent link="FL_calf"/><child link="FL_calflower"/>
+  </joint>
+  <link name="FL_calflower1">
+    <collision><origin xyz="0 0 0"/><geometry><cylinder length="0.03" radius="0.0155"/></geometry></collision>
+  </link>
+  <joint name="FL_calflower1_joint" type="fixed">
+    <origin xyz="-0.01 0 -0.04" rpy="0 0.48 0"/>
+    <parent link="FL_calflower"/><child link="FL_calflower1"/>
+  </joint>
+  <link name="FL_calf_rotor">
+    <inertial><origin xyz="0 0 0"/><mass value="0.089"/><inertia ixx="0.0000596" ixy="0" ixz="0" iyy="0.0001118" iyz="0" izz="0.0000596"/></inertial>
+  </link>
+  <joint name="FL_calf_rotor_joint" type="fixed">
+    <origin xyz="0 -0.03235 0" rpy="0 0 0"/>
+    <parent link="FL_thigh"/><child link="FL_calf_rotor"/>
+  </joint>
+  <link name="FL_foot">
+    <inertial><origin xyz="0 0 0"/><mass value="0.04"/><inertia ixx="9.6E-06" ixy="0" ixz="0" iyy="9.6E-06" iyz="0" izz="9.6E-06"/></inertial>
+    <visual><origin xyz="-0.002 0 0"/><geometry><sphere radius="0.022"/></geometry><material name="matte_black"/></visual>
+    <collision><origin xyz="-0.002 0 0"/><geometry><sphere radius="0.022"/></geometry></collision>
+  </link>
+  <joint name="FL_foot_joint" type="fixed" dont_collapse="true">
+    <origin xyz="0 0 -0.213" rpy="0 0 0"/>
+    <parent link="FL_calf"/><child link="FL_foot"/>
+  </joint>
+  <!-- FR Leg -->
+  <link name="FR_hip">
+    <inertial>
+      <origin xyz="-0.0054 -0.00194 -0.000105" rpy="0 0 0"/><mass value="0.678"/>
+      <inertia ixx="0.00048" ixy="3.01E-06" ixz="1.11E-06" iyy="0.000884" iyz="-1.42E-06" izz="0.000596"/>
+    </inertial>
+    <visual>
+      <origin xyz="0 -0.08 0" rpy="1.5707963 0 0"/><geometry><cylinder length="0.04" radius="0.046"/></geometry>
+      <material name="matte_black"/>
+    </visual>
+    <collision>
+      <origin xyz="0 -0.08 0" rpy="1.5707963 0 0"/><geometry><cylinder length="0.04" radius="0.046"/></geometry>
+    </collision>
+  </link>
+  <joint name="FR_hip_joint" type="revolute">
+    <origin xyz="0.1934 -0.0465 0" rpy="0 0 0"/>
+    <parent link="base"/><child link="FR_hip"/>
+    <axis xyz="1 0 0"/><limit lower="-1.0472" upper="1.0472" effort="95.0" velocity="30.1"/>
+  </joint>
+  <link name="FR_hip_rotor">
+    <inertial><origin xyz="0 0 0"/><mass value="0.089"/><inertia ixx="0.0001118" ixy="0" ixz="0" iyy="0.0000596" iyz="0" izz="0.0000596"/></inertial>
+  </link>
+  <joint name="FR_hip_rotor_joint" type="fixed">
+    <origin xyz="0.11215 -0.04675 0" rpy="0 0 0"/>
+    <parent link="base"/><child link="FR_hip_rotor"/>
+  </joint>
+  <link name="FR_thigh">
+    <inertial>
+      <origin xyz="-0.00374 0.0223 -0.0327" rpy="0 0 0"/><mass value="1.152"/>
+      <inertia ixx="0.00584" ixy="-8.72E-05" ixz="-0.000289" iyy="0.0058" iyz="-0.000808" izz="0.00103"/>
+    </inertial>
+    <visual>
+      <origin xyz="0 0 -0.1065" rpy="0 1.5707963 0"/><geometry><box size="0.213 0.0245 0.034"/></geometry>
+      <material name="matte_black"/>
+    </visual>
+    <collision>
+      <origin xyz="0 0 -0.1065" rpy="0 1.5707963 0"/><geometry><box size="0.213 0.0245 0.034"/></geometry>
+    </collision>
+  </link>
+  <joint name="FR_thigh_joint" type="revolute">
+    <origin xyz="0 -0.0955 0" rpy="0 0 0"/>
+    <parent link="FR_hip"/><child link="FR_thigh"/>
+    <axis xyz="0 1 0"/><limit lower="-1.5708" upper="3.4907" effort="95.0" velocity="30.1"/>
+  </joint>
+  <link name="FR_thigh_rotor">
+    <inertial><origin xyz="0 0 0"/><mass value="0.089"/><inertia ixx="0.0000596" ixy="0" ixz="0" iyy="0.0001118" iyz="0" izz="0.0000596"/></inertial>
+  </link>
+  <joint name="FR_thigh_rotor_joint" type="fixed">
+    <origin xyz="0 0.00015 0" rpy="0 0 0"/>
+    <parent link="FR_hip"/><child link="FR_thigh_rotor"/>
+  </joint>
+  <link name="FR_calf">
+    <inertial>
+      <origin xyz="0.00548 0.000975 -0.115" rpy="0 0 0"/><mass value="0.154"/>
+      <inertia ixx="0.00108" ixy="-3.4E-07" ixz="1.72E-05" iyy="0.0011" iyz="-8.28E-06" izz="3.29E-05"/>
+    </inertial>
+    <visual>
+      <origin xyz="0.01 0 -0.06" rpy="0 -0.2 0"/><geometry><cylinder length="0.12" radius="0.013"/></geometry>
+      <material name="metallic"/>
+    </visual>
+    <collision>
+      <origin xyz="0.01 0 -0.06" rpy="0 -0.2 0"/><geometry><cylinder length="0.12" radius="0.013"/></geometry>
+    </collision>
+  </link>
+  <joint name="FR_calf_joint" type="revolute">
+    <origin xyz="0 0 -0.213" rpy="0 0 0"/>
+    <parent link="FR_thigh"/><child link="FR_calf"/>
+    <axis xyz="0 1 0"/><limit lower="-2.7227" upper="-0.83776" effort="95.0" velocity="15.70"/>
+  </joint>
+  <link name="FR_calflower">
+    <collision><origin xyz="0 0 0"/><geometry><cylinder length="0.065" radius="0.011"/></geometry></collision>
+  </link>
+  <joint name="FR_calflower_joint" type="fixed">
+    <origin xyz="0.020 0 -0.148" rpy="0 0.05 0"/>
+    <parent link="FR_calf"/><child link="FR_calflower"/>
+  </joint>
+  <link name="FR_calflower1">
+    <collision><origin xyz="0 0 0"/><geometry><cylinder length="0.03" radius="0.0155"/></geometry></collision>
+  </link>
+  <joint name="FR_calflower1_joint" type="fixed">
+    <origin xyz="-0.01 0 -0.04" rpy="0 0.48 0"/>
+    <parent link="FR_calflower"/><child link="FR_calflower1"/>
+  </joint>
+  <link name="FR_calf_rotor">
+    <inertial><origin xyz="0 0 0"/><mass value="0.089"/><inertia ixx="0.0000596" ixy="0" ixz="0" iyy="0.0001118" iyz="0" izz="0.0000596"/></inertial>
+  </link>
+  <joint name="FR_calf_rotor_joint" type="fixed">
+    <origin xyz="0 0.03235 0" rpy="0 0 0"/>
+    <parent link="FR_thigh"/><child link="FR_calf_rotor"/>
+  </joint>
+  <link name="FR_foot">
+    <inertial><origin xyz="0 0 0"/><mass value="0.04"/><inertia ixx="9.6E-06" ixy="0" ixz="0" iyy="9.6E-06" iyz="0" izz="9.6E-06"/></inertial>
+    <visual><origin xyz="-0.002 0 0"/><geometry><sphere radius="0.022"/></geometry><material name="matte_black"/></visual>
+    <collision><origin xyz="-0.002 0 0"/><geometry><sphere radius="0.022"/></geometry></collision>
+  </link>
+  <joint name="FR_foot_joint" type="fixed" dont_collapse="true">
+    <origin xyz="0 0 -0.213" rpy="0 0 0"/>
+    <parent link="FR_calf"/><child link="FR_foot"/>
+  </joint>
+  <!-- RL Leg -->
+  <link name="RL_hip">
+    <inertial>
+      <origin xyz="0.0054 0.00194 -0.000105" rpy="0 0 0"/><mass value="0.678"/>
+      <inertia ixx="0.00048" ixy="3.01E-06" ixz="-1.11E-06" iyy="0.000884" iyz="-1.42E-06" izz="0.000596"/>
+    </inertial>
+    <visual>
+      <origin xyz="0 0.08 0" rpy="1.5707963 0 0"/><geometry><cylinder length="0.04" radius="0.046"/></geometry>
+      <material name="matte_black"/>
+    </visual>
+    <collision>
+      <origin xyz="0 0.08 0" rpy="1.5707963 0 0"/><geometry><cylinder length="0.04" radius="0.046"/></geometry>
+    </collision>
+  </link>
+  <joint name="RL_hip_joint" type="revolute">
+    <origin xyz="-0.1934 0.0465 0" rpy="0 0 0"/>
+    <parent link="base"/><child link="RL_hip"/>
+    <axis xyz="1 0 0"/><limit lower="-1.0472" upper="1.0472" effort="95.0" velocity="30.1"/>
+  </joint>
+  <link name="RL_hip_rotor">
+    <inertial><origin xyz="0 0 0"/><mass value="0.089"/><inertia ixx="0.0001118" ixy="0" ixz="0" iyy="0.0000596" iyz="0" izz="0.0000596"/></inertial>
+  </link>
+  <joint name="RL_hip_rotor_joint" type="fixed">
+    <origin xyz="-0.11215 0.04675 0" rpy="0 0 0"/>
+    <parent link="base"/><child link="RL_hip_rotor"/>
+  </joint>
+  <link name="RL_thigh">
+    <inertial>
+      <origin xyz="-0.00374 -0.0223 -0.0327" rpy="0 0 0"/><mass value="1.152"/>
+      <inertia ixx="0.00584" ixy="8.72E-05" ixz="-0.000289" iyy="0.0058" iyz="0.000808" izz="0.00103"/>
+    </inertial>
+    <visual>
+      <origin xyz="0 0 -0.1065" rpy="0 1.5707963 0"/><geometry><box size="0.213 0.0245 0.034"/></geometry>
+      <material name="matte_black"/>
+    </visual>
+    <collision>
+      <origin xyz="0 0 -0.1065" rpy="0 1.5707963 0"/><geometry><box size="0.213 0.0245 0.034"/></geometry>
+    </collision>
+  </link>
+  <joint name="RL_thigh_joint" type="revolute">
+    <origin xyz="0 0.0955 0" rpy="0 0 0"/>
+    <parent link="RL_hip"/><child link="RL_thigh"/>
+    <axis xyz="0 1 0"/><limit lower="-0.5236" upper="4.5379" effort="95.0" velocity="30.1"/>
+  </joint>
+  <link name="RL_thigh_rotor">
+    <inertial><origin xyz="0 0 0"/><mass value="0.089"/><inertia ixx="0.0000596" ixy="0" ixz="0" iyy="0.0001118" iyz="0" izz="0.0000596"/></inertial>
+  </link>
+  <joint name="RL_thigh_rotor_joint" type="fixed">
+    <origin xyz="0 -0.00015 0" rpy="0 0 0"/>
+    <parent link="RL_hip"/><child link="RL_thigh_rotor"/>
+  </joint>
+  <link name="RL_calf">
+    <inertial>
+      <origin xyz="0.00548 -0.000975 -0.115" rpy="0 0 0"/><mass value="0.154"/>
+      <inertia ixx="0.00108" ixy="3.4E-07" ixz="1.72E-05" iyy="0.0011" iyz="8.28E-06" izz="3.29E-05"/>
+    </inertial>
+    <visual>
+      <origin xyz="0.01 0 -0.06" rpy="0 -0.2 0"/><geometry><cylinder length="0.12" radius="0.013"/></geometry>
+      <material name="metallic"/>
+    </visual>
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